File: device/hardware/monolith/monolith.kicad_pcb (KiCad board)
At the start: 2 copper layers, 96 x 74.4 mm, 139 parts, among them J1 CAN, J10 UART, J11 DIN1/2, J12 DIN3/4, J13 Micro_SD_Card, J2 GPS, J3 I2C, J4 AIN1/2, J5 AIN3/4, J6 AIN5/6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

Commit message: update: misc pcb changes
Parts:
- removed J7: USB, Connector_PinHeader_1.00mm:PinHeader_1x02_P1.00mm_Vertical
- moved J2 11.1 mm to (86.7, 148.3)
- moved J3 11.1 mm to (97.8, 148.3)
Connections:
- U2 pad 13: Net-(J7-Pin_1) -> /DBGTX
- U2 pad 14: Net-(J7-Pin_2) -> /DBGRX
- U2 pad 8: /DBGTX -> unconnected-(U2-IO15-Pad8)
- U2 pad 9: /DBGRX -> unconnected-(U2-IO16-Pad9)
Routing:
- net /DBGTX: track 54.6 -> 45.4 mm
- net /GPS_TX: track 47.0 -> 54.0 mm
- net /DBGRX: track 51.3 -> 45.3 mm
- net Net-(J7-Pin_2): track 4.17 -> 0.00 mm
- net Net-(J7-Pin_1): track 4.06 -> 0.00 mm
- net /GPS_RX: track 46.4 -> 50.2 mm
Other:
- board text added: "2.1.0"
- board text removed: "2.0.1"
- board text removed: "D+"
- board text removed: "D-"
