File: device/hardware/monolith/monolith.kicad_sch (KiCad schematic)
At the start: 133 parts, among them J1 CAN, J10 UART, J11 DIN1/2, J12 DIN3/4, J13 Micro_SD_Card, J2 GPS, J3 I2C, J4 AIN1/2, J5 AIN3/4, J6 AIN5/6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

Commit message: update: misc pcb changes
Parts:
- removed J7: USB, Connector_PinHeader_1.00mm:PinHeader_1x02_P1.00mm_Vertical, symbol Connector:Conn_01x02_Pin
Connections:
- net DBGRX: now also U2.14 (USB_D+); no longer U2.9 (IO16)
- net DBGTX: now also U2.13 (USB_D-); no longer U2.8 (IO15)
- no-connect marks 19 -> 21
Changed lines of the file:
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@@
 	)
 	(no_connect
+		(at 99.06 158.75)
+	)
+	(no_connect
 		(at 332.74 224.79)
 	)
@@
 	)
 	(no_connect
+		(at 99.06 161.29)
+	)
+	(no_connect
 		(at 264.16 144.78)
 	)
@@
 	(wire
 		(pts
+			(xy 129.54 128.27) (xy 138.43 128.27)
+		)
+		(stroke
+			(width 0)
+			(type default)
+		)
+	)
+	(wire
+		(pts
 			(xy 116.84 50.8) (xy 118.11 50.8)
 		)
@@
 	(wire
 		(pts
-			(xy 91.44 158.75) (xy 99.06 158.75)
-		)
-		(stroke
-			(width 0)
-			(type default)
-		)
-	)
-	(wire
-		(pts
 			(xy 177.8 44.45) (xy 215.9 44.45)
 		)
@@
 	(wire
 		(pts
-			(xy 91.44 161.29) (xy 99.06 161.29)
-		)
-		(stroke
-			(width 0)
-			(type default)
-		)
-	)
-	(wire
-		(pts
 			(xy 261.62 194.31) (xy 267.97 194.31)
 		)
@@
 	(wire
 		(pts
+			(xy 129.54 125.73) (xy 138.43 125.73)
+		)
+		(stroke
+			(width 0)
+			(type default)
+		)
+	)
+	(wire
+		(pts
 			(xy 104.14 191.77) (xy 104.14 194.31)
 		)
@@
 		)
 	)
-	(label "DBGTX"
-		(at 91.44 158.75 0)
-		(effects
-			(font
-				(size 1.27 1.27)
-			)
-			(justify left bottom)
-		)
-	)
 	(label "TX"
 		(at 138.43 115.57 180)
@@
 		)
 	)
-	(label "DBGRX"
-		(at 91.44 161.29 0)
-		(effects
-			(font
-				(size 1.27 1.27)
-			)
-			(justify left bottom)
-		)
-	)
 	(label "RX"
 		(at 143.51 36.83 0)
@@
 		)
 	)
+	(label "DBGRX"
+		(at 138.43 128.27 180)
+		(effects
+			(font
+				(size 1.27 1.27)
+			)
+			(justify right bottom)
+		)
+	)
 	(label "ADC3"
 		(at 270.51 232.41 0)
@@
 		)
 	)
+	(label "DBGTX"
+		(at 138.43 125.73 180)
+		(effects
+			(font
+				(size 1.27 1.27)
+			)
+			(justify right bottom)
+		)
+	)
 	(label "DIN1"
 		(at 165.1 67.31 180)
@@
 					(unit 1)
 				)
-			)
-		)
-	)
-	(symbol
-		(lib_id "Connector:Conn_01x02_Pin")
-		(at 134.62 125.73 0)
-		(mirror y)
-		(unit 1)
-		(exclude_from_sim no)
-		(in_bom yes)
-		(on_board yes)
-		(dnp no)
-		(property "Reference" "J7"
-			(at 135.636 127 0)
-			(effects
-				(font
-					(size 1.27 1.27)
-				)
-				(justify right)
-				(hide yes)
-			)
-		)
-		(property "Value" "USB"
-			(at 135.636 127 0)
-			(effects
-				(font
-					(size 1.27 1.27)
-				)
-				(justify right)
-			)
-		)
-		(property "Footprint" "Connector_PinHeader_1.00mm:PinHeader_1x02_P1.00mm_Vertical"
-			(at 134.62 125.73 0)
-			(effects
-				(font
-					(size 1.27 1.27)
-				)
-				(hide yes)
-			)
-		)
-		(property "Datasheet" "~"
-			(at 134.62 125.73 0)
-			(effects
-				(font
-					(size 1.27 1.27)
-				)
-				(hide yes)
-			)
-		)
-		(property "Description" "Generic connector, single row, 01x02, script generated"
-			(at 134.62 125.73 0)
-			(effects
-				(font
-					(size 1.27 1.27)
-				)
-				(hide yes)
-			)
-		)
-		(pin "1"
-		)
-		(pin "2"
-		)
-		(instances
-			(project "monolith"
-				(path "/b7db850d-5ff4-4f11-a513-b813e630d63a"
-					(reference "J7")
-					(unit 1)
-				)
