File: device/hardware/monolith-mini/monolith-mini.kicad_pcb (KiCad board)
At the start: 2 copper layers, 51.6 x 74.4 mm, 71 parts, among them J1 PWR/CAN, J10 UART, J13 Micro_SD_Card, J2 GPS, J3 I2C, J4 AUXPWR, Q1 SS8050, Q2 SS8050, U10 LMV321, U11 PCF8563T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

Commit message: update: misc pcb changes
Parts:
- moved J2 11.1 mm to (144.9, 133.0)
- moved J3 11.1 mm to (156.0, 133.0)
- moved R41 1.19 mm to (128.6, 90.2), turned to 0 degrees
- moved R40 1.10 mm to (125.2, 90.2), turned to 180 degrees
- moved J10 0.28 mm to (128.0, 100.1)
- moved C38 0.10 mm to (126.7, 102.7)
- moved D9 0.08 mm to (131.7, 108.2)
Connections:
- U2 pad 13: /DBGRX -> /DBGTX
- U2 pad 14: /DBGTX -> /DBGRX
Routing:
- net /DBGRX: track 40.4 -> 58.0 mm
- net /DBGTX: track 36.8 -> 54.1 mm
- net GND: track 62.8 -> 66.8 mm, vias 35 -> 32
- net /RTS: track 10.8 -> 13.8 mm
- net /GPS_RX: track 51.8 -> 49.0 mm
- net /GPS_TX: track 51.3 -> 49.1 mm
Other:
- board text added: "2.1.0"
- board text removed: "2.0.1"
