File: device/hardware/monolith-mini/monolith-mini.kicad_sch (KiCad schematic)
At the start: 65 parts, among them J1 PWR/CAN, J10 UART, J13 Micro_SD_Card, J2 GPS, J3 I2C, J4 AUXPWR, Q1 SS8050, Q2 SS8050, U10 LMV321, U11 PCF8563T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

Commit message: update: misc pcb changes
Connections:
- net DBGRX: now also U2.14 (USB_D+); no longer U2.13 (USB_D-)
- net DBGTX: now also U2.13 (USB_D-); no longer U2.14 (USB_D+)
Changed lines of the file:
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@@
 		)
 	)
-	(label "DBGRX"
+	(label "DBGTX"
 		(at 140.97 166.37 180)
 		(effects
@@
 		)
 	)
-	(label "DBGTX"
-		(at 140.97 168.91 180)
-		(effects
-			(font
-				(size 1.27 1.27)
-			)
-			(justify right bottom)
-		)
-	)
 	(label "CANTX"
 		(at 93.98 179.07 0)
@@
 		)
 	)
+	(label "DBGRX"
+		(at 140.97 168.91 180)
+		(effects
+			(font
+				(size 1.27 1.27)
+			)
+			(justify right bottom)
+		)
+	)
